File: niu-merged.kicad_pcb (KiCad board)
At the start: 2 copper layers, 241.3 x 103.1 mm, 85 parts

Commit message: add routed merged pcb
Parts:
- moved S22 167.1 mm to (284.9, 152.9)
- moved D18 167.1 mm to (144.0, 149.4)
- moved D39 167.1 mm to (208.1, 149.4)
- moved S21 167.1 mm to (161.1, 168.8)
- moved S42 167.1 mm to (191.1, 168.8)
- moved D12 167.1 mm to (111.3, 96.7)
- moved S1 167.1 mm to (67.2, 152.9)
- moved S20 167.1 mm to (148.5, 107.2)
- moved D15 167.1 mm to (127.7, 122.6)
- moved D24 167.1 mm to (281.4, 119.6)
- moved D38 167.1 mm to (210.1, 168.3)
- moved D20 167.1 mm to (148.0, 111.7)
- moved D27 167.1 mm to (264.2, 137.5)
- moved S41 167.1 mm to (203.7, 107.2)
- moved D16 167.1 mm to (129.7, 103.7)
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Routing:
- net P16: track 0.00 -> 418.6 mm, vias 0 -> 4
- net P4: track 0.00 -> 404.0 mm, vias 0 -> 2
- net P5: track 0.00 -> 371.4 mm, vias 0 -> 1
- net P9: track 0.00 -> 331.5 mm
- net P3: track 0.00 -> 330.2 mm, vias 0 -> 4
- net P8: track 0.00 -> 290.9 mm
- net P2: track 0.00 -> 290.8 mm, vias 0 -> 1
- net P7: track 0.00 -> 261.2 mm, vias 0 -> 2
- net P6: track 0.00 -> 212.6 mm, vias 0 -> 2
- net P10: track 0.00 -> 101.3 mm, vias 0 -> 2
- net mirror_inner_num: track 0.00 -> 15.2 mm
- net mirror_middle_bottom: track 0.00 -> 14.4 mm
- net middle_bottom: track 0.00 -> 14.4 mm
- net index_num: track 0.00 -> 14.4 mm
- net mirror_middle_home: track 0.00 -> 14.4 mm
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- added copper zone on B.Cu, net GND
- added copper zone on F.Cu, net GND
