File: niu-merged.kicad_pcb (KiCad board)
At the start: 2 copper layers, 241.3 x 103.1 mm, 85 parts

Commit message: finalize merged pcb
Parts:
- added G***: LOGO, LOGO, F.Cu at (118.9, 200.5)
- added G***: LOGO, LOGO, F.Cu at (263.1, 200.8)
- moved D15 37.3 mm to (142.7, 156.8)
- moved D18 37.3 mm to (159.0, 183.6)
- moved S21 37.3 mm to (176.1, 203.0)
- moved D9 37.3 mm to (120.4, 187.6)
- moved D24 37.3 mm to (296.4, 153.8)
- moved S12 37.3 mm to (126.8, 126.4)
- moved S27 37.3 mm to (278.7, 167.2)
- moved S9 37.3 mm to (120.9, 183.1)
- moved S3 37.3 mm to (86.2, 149.3)
- moved D17 37.3 mm to (157.0, 202.5)
- moved S25 37.3 mm to (294.0, 130.4)
- moved D5 37.3 mm to (101.0, 190.6)
- moved D16 37.3 mm to (144.7, 137.9)
- moved S28 37.3 mm to (276.8, 148.3)
- moved D39 37.3 mm to (223.2, 183.6)
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Routing:
- net P6: track 212.6 -> 211.8 mm
- net P2: track 290.8 -> 290.1 mm
- net P10: vias 2 -> 1
Other:
- outline, holes or cut-outs redrawn
