File: pcb/jc.kicad_pcb (KiCad board)
At the start: 2 copper layers, 244.7 x 103.8 mm, 105 parts

Commit message: final ver
Parts:
- removed G***: LOGO, LOGO
- moved S31 0.62 mm to (273.5, 167.8)
- moved S34 0.62 mm to (266.6, 111.2)
- moved D39 0.62 mm to (237.7, 187.8)
- moved D14 0.62 mm to (150.2, 160.7)
- moved D43 0.62 mm to (219.7, 197.1)
- moved S42 0.62 mm to (230.2, 126.8)
- moved S22 0.62 mm to (186.8, 173.8)
- moved ? 0.62 mm to (92.4, 163.7)
- moved D18 0.62 mm to (168.3, 169.0)
- moved D21 0.62 mm to (184.0, 197.1)
- moved S29 0.62 mm to (288.4, 132.7)
- moved D38 0.62 mm to (248.9, 123.0)
- moved D31 0.62 mm to (274.1, 172.3)
- moved S21 0.62 mm to (184.5, 192.6)
- moved D32 0.62 mm to (271.8, 153.4)
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Other:
- board text added: "- Koring Doring"
- board text added: "01001000 01000010 01000100 01001010 01000011 01010000 00100001"
- board text added: "Another year closer to the void. May the shadows embrace you with their familiar chill. - Llama 3.1 405B"
- board text added: "Bullseye, bullseye, bullseye! -Matt"
- board text added: "Go placidly amid the noise & haste, & remember what peace there may be in silence. -Lucie"
- board text added: "Happy Birthday JC! Socrates says - {dblquote}He is richest who is content with the least…!{dblquote} Love from Mom and Dad!"
- board text added: "Happy Birthday, JC. Stay fookin' beautiful. -Todd"
- board text added: "It's safe to drink oil in large quantities. The doctors don't want you to know this, but you can do it. Cholesterol is just a number. - mo"
- board text added: "Your PCB does NOT say $cammin, happy birthday! - Jon"
