File: pcb/niu-compact.kicad_pcb (KiCad board)
At the start: 2 copper layers, 245.2 x 104.3 mm, 104 parts

Commit message: [PCB] Add silkscreen, change hatch fill to solid
Parts:
- added G***: LOGO, LOGO, B.Cu at (202.3, 146.6)
- moved ? 30.7 mm to (268.3, 120.9)
- moved ? 30.7 mm to (273.0, 158.6)
- moved D23 30.7 mm to (313.6, 177.8)
- moved D26 30.7 mm to (306.7, 121.2)
- moved D31 30.7 mm to (274.7, 172.5)
- moved D33 30.7 mm to (270.0, 134.8)
- moved S23 30.7 mm to (313.1, 173.3)
- moved S32 30.7 mm to (271.8, 149.2)
- moved S3 30.7 mm to (96.4, 135.6)
- moved D10 30.7 mm to (132.5, 153.6)
- moved D11 30.7 mm to (134.8, 134.8)
- moved D13 30.7 mm to (148.4, 179.8)
- moved D14 30.7 mm to (150.7, 160.9)
- moved D16 30.7 mm to (155.4, 123.2)
- moved D17 30.7 mm to (166.6, 188.0)
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
Commit message: final ver
Other:
- board size 245.2 x 104.3 mm -> 244.7 x 103.8 mm
