File: pcb/niu-v4.kicad_pcb (KiCad board)
At the start: 2 copper layers, 244.7 x 114.2 mm, 106 parts

Commit message: finalize v4
Parts:
- added G***: LOGO, LOGO, B.Cu at (217.6, 158.3)
- added G***: LOGO, LOGO, B.Cu at (211.9, 125.8)
- moved D15 3.62 mm to (162.5, 121.5)
- moved D25 3.62 mm to (318.4, 119.5)
- moved S19 3.62 mm to (181.1, 125.3)
- moved S44 3.62 mm to (226.8, 153.4)
- moved ? 3.62 mm to (277.7, 100.3)
- moved D20 3.62 mm to (182.9, 110.9)
- moved D30 3.62 mm to (296.6, 98.0)
- moved D5 3.62 mm to (120.1, 154.6)
- moved D7 3.62 mm to (124.7, 116.9)
- moved D4 3.62 mm to (107.6, 100.7)
- moved ? 3.62 mm to (246.0, 153.6)
- moved D13 3.62 mm to (157.8, 159.2)
- moved ? 3.62 mm to (107.0, 105.6)
- moved D28 3.62 mm to (301.2, 135.7)
- moved D23 3.62 mm to (323.0, 157.2)
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Routing:
- net B2: track 0.00 -> 415.3 mm, vias 0 -> 4
- net B3: track 0.00 -> 373.4 mm, vias 0 -> 4
- net E6: track 0.00 -> 365.6 mm, vias 0 -> 2
- net B4: track 0.00 -> 315.6 mm, vias 0 -> 1
- net D1: track 0.00 -> 198.1 mm, vias 0 -> 1
- net F4: track 0.00 -> 186.2 mm, vias 0 -> 1
- net D0: track 0.00 -> 171.9 mm, vias 0 -> 1
- net F5: track 0.00 -> 163.0 mm, vias 0 -> 1
- net D2: track 0.00 -> 145.6 mm, vias 0 -> 2
- net D4: track 0.00 -> 145.1 mm, vias 0 -> 1
- net B6: track 0.00 -> 144.5 mm, vias 0 -> 4
- net D3: track 0.00 -> 141.6 mm, vias 0 -> 2
- net F6: track 0.00 -> 135.8 mm, vias 0 -> 1
- net C6: track 0.00 -> 122.5 mm, vias 0 -> 1
- net F7: track 0.00 -> 114.6 mm, vias 0 -> 1
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- added copper zone on B.Cu, net GND
- added copper zone on F.Cu, net GND
